File: hardware/kicad/wigglecam.kicad_pcb (KiCad board)
At the start: 4 copper layers, 76 x 50 mm, 105 parts, among them J1 SWD, J2 USB-C, J3 LED1, J4 LED2, J5 VBAT_IN, J6 VBAT_OUT, J7 SHUTTER, J8 Pi GPIO 1-12, Q1 AO3401A, Q2 AO3400A, Q3 AO3400A, SW1 TACT, SW2 TACT, SW3 EC11, U1 AP2112K-3.3, U2 RP2040, U3 W25Q128JVSIQ, U4 USBLC6-2SC6, U5 LM358, U6 INA219, Y1 12MHz

Commit message: Re-route the board by hand; drop the scripted layout pipeline
Lay the signal routing out in KiCad by hand: the critical nets
(RP2040 fan-out, QSPI flash bus, USB differential pair, crystal,
flash-current loop, power entry and battery path) routed first, then
the low-speed GPIO worked in around them, kept off the inner GND and
3V3/VLED planes. Board is fully routed and DRC-clean (0 violations,
0 unconnected); the 24-check measured verification pass has no FAILs,
including the flash-path copper-width check.

Remove the generative placement/routing pipeline
(hardware/scripts/01-05*), the Freerouting round-trip artifacts
(wigglecam.dsn/.ses and freerouting.log), and the pipeline plan doc.
Keep the fab-export, DRC, and verification helpers. Regenerate the
gerbers, drill, renders, and DRC report from the re-routed board and
reword the README and docs to describe the hand layout.

Keep the Python tooling out of the repository language stats via
.gitattributes.
Routing:
- net WS_VDD: track 33.6 -> 25.1 mm, vias 0 -> 2
- net N$12: track 37.6 -> 44.1 mm
- net WS_DIN_R: track 29.3 -> 35.4 mm
- net N$6: track 13.9 -> 19.5 mm, vias 0 -> 2
- net VSYS: track 82.5 -> 87.0 mm, vias 2 -> 9
- net SHUTTER_RAW: track 29.0 -> 25.9 mm, vias 1 -> 2
- net UART_RX_HDR: track 16.0 -> 18.1 mm, vias 0 -> 1
- net N$8: track 8.65 -> 7.00 mm, vias 0 -> 2
- net N$5: track 7.04 -> 5.96 mm
- net N$9: track 5.18 -> 4.18 mm
- net ENC_B_RAW: track 20.6 -> 21.4 mm
- net SPARE_IO_HDR: track 15.9 -> 16.7 mm, vias 0 -> 1
- net CAM_SYNC_HDR: track 11.7 -> 11.0 mm
- net ENC_SW1_RAW: track 16.9 -> 17.5 mm
