File: hardware/kicad/wigglecam.kicad_pcb (KiCad board)
At the start: 4 copper layers, 76 x 50 mm, 105 parts, among them J1 SWD, J2 USB-C, J3 LED1, J4 LED2, J5 VBAT_IN, J6 VBAT_OUT, J7 SHUTTER, J8 Pi GPIO 1-12, Q1 AO3401A, Q2 AO3400A, Q3 AO3400A, SW1 TACT, SW2 TACT, SW3 EC11, U1 AP2112K-3.3, U2 RP2040, U3 W25Q128JVSIQ, U4 USBLC6-2SC6, U5 LM358, U6 INA219, Y1 12MHz

Commit message: Board fully routed, DRC clean: 0 errors, 0 unconnected (JLCPCB 4-layer rules)
Hybrid flow as planned: scripted critical nets (QSPI nested lanes,
crystal, USB differential pair with mirror-pad B.Cu jumpers, power
entry, battery path, LED returns, plane fanout stubs and QFN interior
power fanouts), Freerouting 1.9 for the low-speed remainder (inner
plane layers marked unroutable, completed nets stripped from the DSN,
outline shrunk for edge clearance), zone pours with island removal,
then scripted finishing passes closing the final airwires with
collision-checked geometry (05_finish through 05i, incl. a dual-layer
BFS maze route for the ENC_A leg). The full DRC gate runs kicad-cli
with refilled zones at every step.
Parts:
- D5: value 1N4148WS -> 1N4148W; footprint D_SOD-323 -> D_SOD-123
- moved R4 29.7 mm to (115.8, 118.8)
- moved R33 29.1 mm to (143.7, 112.6)
- moved C22 26.9 mm to (129.7, 142.3)
- moved C18 26.4 mm to (129.8, 145.2)
- moved C33 24.8 mm to (133.4, 135.9)
- moved R11 21.7 mm to (148.5, 131.0)
- moved R32 21.5 mm to (115.3, 106.4)
- moved C34 13.3 mm to (129.9, 137.3)
- moved C24 13.2 mm to (144.4, 132.1)
- moved C5 12.4 mm to (113.2, 125.8)
- moved R10 11.0 mm to (142.3, 130.0)
- moved R12 9.51 mm to (152.8, 132.5)
- moved FID3 8.35 mm to (174.0, 108.0)
- moved C16 7.48 mm to (137.3, 106.8)
- moved R29 7.11 mm to (170.8, 102.1)
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Connections:
- D4 pad 2: __NOCONNECT -> (no net)
- J2 pad A8: __NOCONNECT -> (no net)
- J2 pad B8: __NOCONNECT -> (no net)
- J8 pad 1: __NOCONNECT -> (no net)
- J8 pad 7: __NOCONNECT -> (no net)
- SW1 pad 2: __NOCONNECT -> (no net)
- SW1 pad 3: __NOCONNECT -> (no net)
- SW2 pad 2: __NOCONNECT -> (no net)
- SW2 pad 3: __NOCONNECT -> (no net)
- U2 pad 11: __NOCONNECT -> (no net)
- U2 pad 12: __NOCONNECT -> (no net)
- U2 pad 17: __NOCONNECT -> (no net)
- U2 pad 18: __NOCONNECT -> (no net)
- U2 pad 28: __NOCONNECT -> (no net)
- U2 pad 29: __NOCONNECT -> (no net)
- U2 pad 30: __NOCONNECT -> (no net)
- U2 pad 31: __NOCONNECT -> (no net)
- U2 pad 32: __NOCONNECT -> (no net)
- U2 pad 35: __NOCONNECT -> (no net)
- U2 pad 36: __NOCONNECT -> (no net)
- U2 pad 38: __NOCONNECT -> (no net)
- U2 pad 39: __NOCONNECT -> (no net)
- U2 pad 40: __NOCONNECT -> (no net)
- U2 pad 41: __NOCONNECT -> (no net)
Routing:
- net VSYS: track 0.00 -> 82.5 mm, vias 0 -> 2
- net ENC_A: track 0.00 -> 82.0 mm, vias 0 -> 9
- net ENC_SW1: track 0.00 -> 76.1 mm, vias 0 -> 3
- net +3V3: track 0.00 -> 68.7 mm, vias 0 -> 36
- net VREG_1V1: track 0.00 -> 62.2 mm, vias 0 -> 6
- net RUN: track 0.00 -> 62.1 mm, vias 0 -> 3
- net ENC_B: track 0.00 -> 54.5 mm, vias 0 -> 3
- net GND: track 5.00 -> 58.6 mm, vias 13 -> 78
- net PI_SCL: track 0.00 -> 41.2 mm, vias 0 -> 2
- net VBUS: track 0.00 -> 40.5 mm
- net I2C0_SDA: track 0.00 -> 39.6 mm
- net N$12: track 0.00 -> 37.6 mm, vias 0 -> 2
- net N$2: track 0.00 -> 34.7 mm, vias 0 -> 1
- net WS_VDD: track 0.00 -> 33.6 mm
- net SPARE_IO: track 0.00 -> 32.7 mm, vias 0 -> 2
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- added copper zone on B.Cu, net GND
- added copper zone on F.Cu, net GND

Commit message: BOM: verified LCSC numbers for every SMT line; order-readiness audit
- Generic R/C lines get concrete LCSC picks (each number verified
  against its LCSC product page for value + package, 2026-07-03);
  resistors are JLC-basic UNI-ROYAL 0603WAF parts.
- USB series Rs changed 27.4R -> 27R (guide-nominal; equivalent at
  USB-FS) so R2/R7/R8 share the basic part C25190. Board Value
  fields, netlist, BOM and CPL regenerated; positions/rotations
  byte-identical, ERC and DRC re-run clean (0/0).
- 470 uF reservoir resolved to Panasonic 6TPE470MI POSCAP (C402828,
  18 mOhm) per the checklist's ESR requirement.
- JST shells pinned to genuine B2B-XH-A (C158012); SWD header and
  2x6 Pi socket left unmatched on purpose (THT hand-solder).
- partlist.md refdes corrected to match the routed board; documented
  the BOOTSEL missing-1k deviation from the reference design in the
  review checklist; gerber zip added for one-click JLCPCB upload.
Parts:
- R7, R8: value 27.4R -> 27R
Changed lines of the file:
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@@
 			)
 		)
-		(property "Value" "27.4R"
+		(property "Value" "27R"
 			(at 0 1.43 90)
 			(layer "F.Fab")
@@
 			)
 		)
-		(property "Value" "27.4R"
+		(property "Value" "27R"
 			(at 0 1.43 90)
 			(layer "F.Fab")

Commit message: Trigger semantics: sync edge always arrives; R12 value propagated
- STATUS bit0 now covers any trigger-engine activity (flash or sync
  pulse), and a TRIGGER=2 refused by the 800 ms cooldown degrades to a
  sync-only pulse instead of vanishing - the Pi's capture loop can no
  longer hang waiting for an edge that never comes. flash_fire()
  reports refusal so the dispatcher can fall back.
- ws2812 writes drop on a full FIFO instead of blocking (reachable
  from the I2C IRQ; at 800 kbit the FIFO drains in ~30 us).
- R12 1.18k propagated to the remaining artifacts: cpl.csv, the
  committed netlist, and the board file's value field; bom.csv row
  order matches regeneration.
- protocol.md: cooldown degrade + high-byte-read latch behavior
  documented; partlist/README claims scoped to the one pending pick.
Parts:
- R12: value 1k -> 1.18k
Changed lines of the file:
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@@
 			)
 		)
-		(property "Value" "1k"
+		(property "Value" "1.18k"
 			(at 0 1.43 0)
 			(layer "F.Fab")

Commit message: R12 to 1.2 k, and split the JLC upload set from the hand-solder parts
The E96 1.18 k is the exact fit for the flash reference divider but is
thinly stocked. 1.2 k settles at 0.508 V instead of 0.5005 V, so
1.015 A per branch instead of 1.001 A. The sense resistor sees 0.515 W
against a 1 W part for at most 150 ms and the sinks are unchanged, so
the 1.5 % costs nothing and the part is a common value. Changed in the
schematic source, netlist, board, BOM, CPL and the docs that quote the
divider math. Copper is untouched: DRC still 0 violations, 0
unconnected.

fab/jlc/ now holds the exact upload set, 90 surface-mount placements
with the eight through-hole parts split into their own list, so the
BOM tool has nothing to reject.
Parts:
- R12: value 1.18k -> 1.2k
Changed lines of the file:
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@@
 			)
 		)
-		(property "Value" "1.18k"
+		(property "Value" "1.2k"
 			(at 0 1.43 0)
 			(layer "F.Fab")
